Commit message: Add wrist-mounted D435 camera and mounting kit

File: src/tactile_robot_description/urdf/xarm6_ag95.urdf.xacro (robot description, xacro)
@@ -3,4 +3,7 @@
   <xacro:arg name="mount_xyz" default="0 0 0"/>
   <xacro:arg name="mount_rpy" default="0 0 0"/>
+  <xacro:arg name="add_camera" default="true"/>
+  <xacro:arg name="camera_mount_xyz" default="0 0 0"/>
+  <xacro:arg name="camera_mount_rpy" default="0 0 0"/>
   <xacro:property name="mesh_suffix" value="stl"/>
   <xacro:property name="mesh_path" value="package://xarm_description/meshes"/>
@@ -10,4 +13,5 @@
   <xacro:include filename="$(find xarm_description)/urdf/xarm6/xarm6.urdf.xacro"/>
   <xacro:include filename="$(find dh_ag95_description)/urdf/dh_ag95_macro.xacro"/>
+  <xacro:include filename="$(find xarm_description)/urdf/camera/realsense_d435i.urdf.xacro"/>
   <xacro:common_material prefix=""/>
   <link name="world"/>
@@ -27,3 +31,18 @@
     <origin xyz="$(arg mount_xyz)" rpy="$(arg mount_rpy)"/>
   </xacro:dh_ag95_gripper>
+  <xacro:if value="$(arg add_camera)">
+    <xacro:common_material prefix="d435_"/>
+    <!-- The upstream macro uses the D435 camera-and-stand STL. Its legacy
+         name contains d435i, but it defines no IMU links or sensors. -->
+    <link name="camera_mount_link"/>
+    <joint name="camera_mount_joint" type="fixed">
+      <parent link="link_eef"/><child link="camera_mount_link"/>
+      <origin xyz="$(arg camera_mount_xyz)" rpy="$(arg camera_mount_rpy)"/>
+    </joint>
+    <xacro:d435i_urdf prefix="d435_" add_d435i_links="true"/>
+    <joint name="camera_kit_joint" type="fixed">
+      <parent link="camera_mount_link"/><child link="d435_link_eef"/>
+      <origin xyz="0 0 0" rpy="0 0 0"/>
+    </joint>
+  </xacro:if>
 </robot>

Commit message: Add UFACTORY 850 as default selectable robot arm

File: src/tactile_robot_description/urdf/xarm6_ag95.urdf.xacro (robot description, xacro)
@@ -1,4 +1,5 @@
 <?xml version="1.0"?>
-<robot name="xarm6_ag95" xmlns:xacro="http://ros.org/wiki/xacro">
+<robot name="tactile_arm_ag95" xmlns:xacro="http://ros.org/wiki/xacro">
+  <xacro:arg name="robot_model" default="uf850"/>
   <xacro:arg name="mount_xyz" default="0 0 0"/>
   <xacro:arg name="mount_rpy" default="0 0 1.5707963267948966"/>
@@ -12,4 +13,5 @@
   <xacro:include filename="$(find xarm_description)/urdf/common/common.link.xacro"/>
   <xacro:include filename="$(find xarm_description)/urdf/xarm6/xarm6.urdf.xacro"/>
+  <xacro:include filename="$(find xarm_description)/urdf/uf850/uf850.urdf.xacro"/>
   <xacro:include filename="$(find dh_ag95_description)/urdf/dh_ag95_macro.xacro"/>
   <xacro:include filename="$(find xarm_description)/urdf/camera/realsense_d435i.urdf.xacro"/>
@@ -20,6 +22,13 @@
     <origin xyz="0 0 0" rpy="0 0 0"/>
   </joint>
-  <xacro:xarm6_urdf prefix=""
-    kinematics_params_filename="$(find xarm_description)/config/kinematics/default/xarm6_default_kinematics.yaml"/>
+  <xacro:property name="selected_model" value="$(arg robot_model)"/>
+  <xacro:if value="${selected_model == 'xarm6'}">
+    <xacro:xarm6_urdf prefix=""
+      kinematics_params_filename="$(find xarm_description)/config/kinematics/default/xarm6_default_kinematics.yaml"/>
+  </xacro:if>
+  <xacro:if value="${selected_model == 'uf850'}">
+    <xacro:uf850_urdf prefix=""
+      kinematics_params_filename="$(find xarm_description)/config/kinematics/default/uf850_default_kinematics.yaml"/>
+  </xacro:if>
   <!-- UFACTORY's nominal tool frame coincides with link6. -->
   <link name="link_eef"/>

Commit message: Add robot-adapted tabletop scene and external camera

File: src/tactile_robot_description/urdf/xarm6_ag95.urdf.xacro (robot description, xacro)
@@ -2,4 +2,5 @@
 <robot name="tactile_arm_ag95" xmlns:xacro="http://ros.org/wiki/xacro">
   <xacro:arg name="robot_model" default="uf850"/>
+  <xacro:arg name="base_xyz" default="0 0 0"/>
   <xacro:arg name="mount_xyz" default="0 0 0"/>
   <xacro:arg name="mount_rpy" default="0 0 1.5707963267948966"/>
@@ -20,5 +21,5 @@
   <joint name="world_joint" type="fixed">
     <parent link="world"/><child link="link_base"/>
-    <origin xyz="0 0 0" rpy="0 0 0"/>
+    <origin xyz="$(arg base_xyz)" rpy="0 0 0"/>
   </joint>
   <xacro:property name="selected_model" value="$(arg robot_model)"/>
